File: texboard_hw_mk2/texboard.brd (EAGLE design)
At the start: 364.5 x 114.7 mm, 200 parts

Commit message: idk
Routing:
- net N$37: track 0.00 -> 26.7 mm
- net GND: track 0.00 -> 16.7 mm
Other:
- board text added: "TIAK mk2 lysandrou2018"
- board text removed: "TeXbrd mk2 lysandrou2018"
