File: texboard_hw_mk2/texboard.sch (EAGLE design)
At the start: 200 parts, among them SW1 CHERRY_MX_STABILIZER_2X, SW2 CHERRY_MX_WITH_FIXING_PINS_&_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, SW3 CHERRY_MX_STABILIZER_2X, SW4 CHERRY_MX_STABILIZER_2X, SW5 CHERRY_MX_STABILIZER_2X, SW6 CHERRY_MX_STABILIZER_2X

Commit message: idk
Other:
- moved on the sheet: H1, H2, H3, H5, H6, H7, H8, U$38
